File: hardware/amp1.sch (KiCad schematic (older format))
At the start: 64 parts, among them Q1 PN2222A, Q10 PN2222A, Q11 PN2222A, Q12 PN2222A, Q13 PN2222A, Q14 PN2222A, Q15 PN2222A, Q16 PN2222A, Q17 PN2222A, Q18 PN2222A, Q19 PN2222A, Q2 PN2222A, Q20 PN2222A, Q21 PN2222A, Q22 PN2222A, Q23 PN2222A, Q24 PN2222A, Q25 PN2222A, Q26 PN2222A, Q27 PN2222A, Q28 PN2222A, Q29 PN2222A, Q3 PN2222A, Q30 PN2222A, Q31 PN2222A, Q32 IRF540N, Q4 PN2222A, Q5 PN2222A, Q6 PN2222A, Q7 PN2222A, Q8 PN2222A, Q9 PN2222A

Commit message: Added PDF and PNG images of the design.
Other:
- note added: "Amplifier circuit for 15 +1 LED strips."
- note removed: "Amplifier circuit for 15+1 RGB LED strips."
Changed lines of the file:
@@
 $EndComp
 Text Notes 7350 7550 0    60   ~ 0
-Amplifier circuit for 15+1 RGB LED strips.
+Amplifier circuit for 15 +1 LED strips.
 $EndSCHEMATC
